File: hw/CAD/iotkit-esp32.brd (EAGLE design)
At the start: 91.1 x 69.8 mm, 4 parts

Commit message: Inkl. Stepper
Parts:
- added (+)STEPPER1: PB0-3, pinhead:1X05
- added (+)STEPPER2: PB4-7, pinhead:1X05
- added (+)STEPPER3: PA7-4, pinhead:1X05
- added 10K: (no value), rcl:0204/7
- added IC1: MCP23017SP 0x20, microchip:DIL28-3
- added S1: PA0, pinhead:1X02
- added S2: PA1, pinhead:1X02
- added S3: PA2, pinhead:1X02
- added STEPPER1, STEPPER2: (no value), SparkFun-IC-Special-Function:DIL18
Connections:
- new net +5V: (+)STEPPER1.1, (+)STEPPER2.1, (+)STEPPER3.1, STEPPER1.10, STEPPER2.10
- new net N$1: (+)STEPPER2.2, STEPPER1.14
- new net N$2: (+)STEPPER2.3, STEPPER1.13
- new net N$3: (+)STEPPER2.4, STEPPER1.12
- new net N$30: (+)STEPPER1.2, STEPPER1.18
- new net N$31: (+)STEPPER1.3, STEPPER1.17
- new net N$32: (+)STEPPER1.4, STEPPER1.16
- new net N$33: (+)STEPPER1.5, STEPPER1.15
- new net N$4: (+)STEPPER2.5, STEPPER1.11
- new net N$5: 10K.2, IC1.18
- new net N$6: (+)STEPPER3.2, STEPPER2.18
- new net N$7: (+)STEPPER3.3, STEPPER2.17
- new net N$8: (+)STEPPER3.4, STEPPER2.16
- new net N$9: (+)STEPPER3.5, STEPPER2.15
- new net PA0: IC1.21, S1.1
- new net PA1: IC1.22, S2.1
- new net PA2: IC1.23, S3.1
- new net PA4: IC1.25, STEPPER2.4
- new net PA5: IC1.26, STEPPER2.3
- new net PA6: IC1.27, STEPPER2.2
- new net PA7: IC1.28, STEPPER2.1
- new net PB0: IC1.1, STEPPER1.1
- new net PB1: IC1.2, STEPPER1.2
- new net PB2: IC1.3, STEPPER1.3
- new net PB3: IC1.4, STEPPER1.4
- new net PB4: IC1.5, STEPPER1.5
- new net PB5: IC1.6, STEPPER1.6
- new net PB6: IC1.7, STEPPER1.7
- new net PB7: IC1.8, STEPPER1.8
- net 3V3: now also 10K.1, IC1.9
- net GND: now also IC1.10, IC1.15, IC1.16, IC1.17, S1.2, S2.2, S3.2, STEPPER1.9, STEPPER2.9
- net SCL: now also IC1.12
- net SDA: now also IC1.13
Other:
- board size 91.1 x 69.8 mm -> 87.3 x 69.8 mm

Commit message: Pos
Parts:
- moved (+)STEPPER1 3.81 mm to (25.4, 68.6)
- moved (+)STEPPER2 3.81 mm to (40.6, 68.6)
- moved (+)STEPPER3 3.81 mm to (55.9, 68.6)
- moved S1 3.81 mm to (67.3, 68.6)
- moved S2 3.81 mm to (74.9, 68.6)
- moved S3 3.81 mm to (82.5, 68.6)
- moved BUZZER 3.81 mm to (10.2, 64.8), turned to 180 degrees
Other:
- board size 87.3 x 69.8 mm -> 87.3 x 72.4 mm
